File: drone/drone.kicad_pcb (KiCad board)
At the start: 2 copper layers, 46 x 46 mm, 65 parts, among them Q1 AO3400A, U2 MPU-6050, U3 MP2303ADN, U4 AMS1117-3.3

Commit message: 6/6
Parts:
- added TP13: TestPoint, TestPoint:TestPoint_Pad_D1.0mm, F.Cu at (85.0, 60.5)
- added TP14: TestPoint, TestPoint:TestPoint_Pad_D1.0mm, B.Cu at (85.0, 60.5)
- added TP15: TestPoint, TestPoint:TestPoint_Pad_D1.0mm, F.Cu at (93.0, 72.3)
- added TP16: TestPoint, TestPoint:TestPoint_Pad_D1.0mm, F.Cu at (93.0, 69.8)
- added TP17: TestPoint, TestPoint:TestPoint_Pad_D1.0mm, F.Cu at (93.0, 74.8)
- C10: value 10nF -> 100nF
- C12: value 22nF -> 10uF
- C5: value 220pF -> 0.1uF
- C6: value 220pF -> 2.2nF
- D1: moved to F.Cu
- moved D1 5.56 mm to (104.1, 88.9), turned to 90 degrees
- moved G*** 1.58 mm to (104.5, 92.0)
- moved TP10 1.50 mm to (87.5, 60.5)
- moved TP11 1.50 mm to (90.0, 60.5)
- moved TP12 1.50 mm to (92.5, 60.5)
- moved TP4 1.50 mm to (90.0, 60.5)
- moved TP5 1.50 mm to (92.5, 60.5)
- moved TP7 1.50 mm to (87.5, 60.5)
Connections:
- +Buzzer1 pad 1: +3V3 -> +5V
- U1 pad 3: unconnected-(U1-GP3-Pad3) -> GPIO3
- U1 pad 4: unconnected-(U1-GP4-Pad4) -> GPIO4
- U1 pad 5: unconnected-(U1-GP5-Pad5) -> GPIO5
Routing:
- net +5V: track 64.7 -> 110.8 mm, vias 3 -> 4
- net ESC VCC: track 141.3 -> 162.3 mm
- net GND: track 18.9 -> 26.6 mm, vias 23 -> 22
- net Net-(D1-A): track 2.30 -> 8.09 mm, vias 0 -> 1
- net GPIO4: track 0.00 -> 3.48 mm
- net +3V3: track 56.9 -> 53.6 mm, vias 1 -> 0
- net GPIO3: track 0.00 -> 3.16 mm
- net GPIO5: track 0.00 -> 3.13 mm
- net TX2: track 11.6 -> 9.78 mm
- net TX1: track 8.99 -> 7.28 mm
- net RX2: track 8.02 -> 6.52 mm
- net SDA: track 27.6 -> 28.9 mm
- net unconnected-(U1-3V3(OUT)-Pad3V3): track 0.00 -> 1.06 mm
- net RX1: track 5.69 -> 4.88 mm
- net SCL: track 26.2 -> 26.8 mm
Other:
- board text added: "3"
- board text added: "4"
- board text added: "5"
- board text added: "5V"
- board text added: "GPIO"
- board text added: "LED 3v3"
