File: drone/drone.kicad_pcb (KiCad board)
At the start: 2 copper layers, 46 x 46 mm, 70 parts, among them Q1 AO3400A, U2 MPU-6050, U3 MP2303ADN, U4 AMS1117-3.3

Commit message: 3/7
Parts:
- moved Q1 11.4 mm to (112.3, 72.4)
- moved C14 0.60 mm to (90.6, 92.4)
- moved TP15 0.40 mm to (92.6, 72.3)
- moved TP16 0.40 mm to (92.6, 69.8)
- moved TP17 0.40 mm to (92.6, 74.8)
- moved -Buzzer1 0.22 mm to (123.1, 67.7)
Routing:
- net /Buzzer: track 16.7 -> 0.00 mm
- net +5V: track 110.8 -> 109.5 mm
- net GND: vias 22 -> 21
